Commit message: Updated Inertias

File: assets/wxai_follower.urdf (robot description, URDF)
Before this commit: robot wxai, 14 links, 13 joints
Links:
- link camera_link: geometry collision box size=0.023 0.042 0.042; visual mesh filename=package://trossen_arm_description/meshes/peripherals/d405.s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 scale=0.001 0.001 0.001
