Commit message: changes

File: trossen_arm_mujoco/assets/wxai_follower.urdf (robot description, URDF)
Before this commit: robot wxai, 14 links, 13 joints
Links:
- removed link camera_bottom_screw_frame
- removed link camera_link
- added link cam_bottom_screw_frame
- added link cam_link, mass 0.072; collision box size=0.023 0.042 0.042; visual mesh filename=package://trossen_arm_description/meshes/peripherals/d405.s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 scale=0.001 0.001 0.001
Joints:
- removed joint camera_joint
- removed joint camera_link_joint
- removed joint camera_mount_joint
- added joint cam_joint: type fixed, parent camera_mount_d405, child cam_bottom_screw_frame, origin xyz=0.02927207801 0 0.03824951197 rpy=0 0.3490658503988659 0
- added joint cam_link_joint: type fixed, parent cam_bottom_screw_frame, child cam_link, origin xyz=0.01085 0.009 0.021 rpy=0 0 0
- added joint cam_mount_joint: type fixed, parent link_6, child camera_mount_d405, origin xyz=0 0 0 rpy=0 0 0, axis 0 0 0
